File: minM3car.brd (EAGLE design)
At the start: 30 x 50.1 mm, 38 parts, among them Q1 BSS84, U1 QRE1113SMD-W, U2 DRV8835

Commit message: nuevo avance
Parts:
- removed JP3: (no value), adafruit:1X03
- added J1: (no value), SparkFun-Connectors:1X02
- R4: value 2k -> 220
- moved U$5 23.9 mm to (20.5, 31.8), turned to 180 degrees
- moved U$7 17.7 mm to (17.8, 21.1), turned to 270 degrees
- moved R7 17.4 mm to (6.70, 18.3)
- moved C3 13.4 mm to (6.10, 10.9), turned to 0 degrees
- moved U$6 12.8 mm to (23.2, 24.6), turned to 90 degrees
- moved J2 8.60 mm to (3.40, 2.20)
- moved U2 8.34 mm to (5.06, 7.88)
- moved R13 6.61 mm to (7.20, 32.4)
- moved D5 5.26 mm to (19.4, 16.2), turned to 180 degrees
- moved U$3 4.88 mm to (2.00, 8.70), turned to 270 degrees
- moved R5 4.47 mm to (27.1, 6.10)
- moved R1 3.98 mm to (7.20, 31.0), turned to 180 degrees
- moved U$1 2.43 mm to (20.5, 22.8), turned to 180 degrees
- moved R8 1.97 mm to (26.9, 43.6), turned to 0 degrees
- moved U1 1.79 mm to (10.6, 17.0), flipped to the bottom
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Connections:
- new net GPIO1: JP1.6, U$2.P0.02
- new net GPIO2: JP1.5, U$2.P0.28
- new net GPIO3: JP1.4, U$2.P0.29
- new net GPIO4: JP1.3, U$2.P0.30
- new net LED1: R8.1, U$2.P0.03
- new net LED2: R9.1, U$2.P1.04
- new net N$11: U$2.P1.03
- new net N$14: U$2.P1.00
- new net N$16: U$2.P0.22
- new net N$17: JP2.3
- new net N$18: JP2.4
- new net N$19: U$2.P1.15
- new net N$22: U$2.P1.13
- new net N$23: U$2.P1.11
- new net N$24: JP2.5
- new net N$25: U$2.P1.02
- new net N$26: U$2.P1.01
- new net N$27: U$2.P0.04
- new net N$28: U$2.P0.05
- new net N$29: U$2.P0.10
- new net N$30: U$2.P0.31
- new net N$31: JP2.6
- net GND: now also J1.2, JP1.1
- net N$10: now also U$2.P1.06; no longer JP3.3
- net N$4: now also U$2.P0.21; no longer JP3.1
- net N$5: now also JP2.1; no longer R8.1
- net N$6: now also JP2.2; no longer R9.1
- net N$7: now also U$2.P0.09; no longer JP3.2
- net VBAT: now also J1.1
- net VCC: now also JP1.2; no longer U2.1
- net VSUPL: now also U2.1
Routing:
- net VBAT: track 0.00 -> 54.3 mm, vias 0 -> 4
- net VCC: track 0.00 -> 46.2 mm, vias 0 -> 2
- net VBUS: track 0.00 -> 34.2 mm, vias 0 -> 3
- net D-: track 0.00 -> 27.2 mm, vias 0 -> 2
- net D+: track 0.00 -> 26.2 mm
- net VSUPL: track 0.00 -> 13.3 mm
- net GPIO4: track 0.00 -> 11.0 mm
- net GPIO3: track 0.00 -> 9.45 mm
- net GPIO2: track 0.00 -> 7.21 mm
- net GPIO1: track 0.00 -> 6.62 mm
- net N$2: track 0.00 -> 6.49 mm, vias 0 -> 2
- net LED2: track 0.00 -> 6.48 mm
- net N$9: track 0.00 -> 4.12 mm
- net N$8: track 0.00 -> 4.02 mm
- net LED1: track 0.00 -> 3.86 mm
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- added copper zone on layer 1, net GND
- added copper zone on layer 16, net GND

Commit message: nuevo avance
Parts:
- D2: value (none) -> 200mA/100V/1V; device SparkFun-DiscreteSemi:SOD-323@1 -> SparkFun-DiscreteSemi:DIODE-1N4148
- U1: value QRE1113SMD-W -> (none)
- moved R12 50.7 mm to (10.1, 12.2)
- moved Q1 44.2 mm to (10.5, 7.30)
- moved R1 7.21 mm to (14.4, 31.3), turned to 270 degrees
- moved R13 5.51 mm to (12.6, 31.3), turned to 90 degrees
- moved R10 4.53 mm to (-29.8, -13.9)
- moved U$4 0.73 mm to (2.30, 11.1)
- moved U$3 0.57 mm to (1.60, 9.10)
Connections:
- removed net N$14: U$2.P1.00
- removed net N$17: JP2.3
- removed net N$18: JP2.4
- removed net N$24: JP2.5
- removed net N$25: U$2.P1.02
- removed net N$26: U$2.P1.01
- removed net N$31: JP2.6
- new net GPIO5: JP2.6, U$2.P1.02
- new net GPIO6: JP2.5, U$2.P1.01
- new net GPIO7: JP2.4, U$2.P1.03
- new net GPIO8: JP2.3, U$2.P1.00
- net GND: now also JP2.1
- net N$11: now also U$2.P0.19; no longer U$2.P1.03
- net N$12: now also D2.A; no longer D2.2
- net N$5: now also U$2.P0.23; no longer JP2.1
- net N$6: now also U$2.P0.12; no longer JP2.2
- net VCC: now also JP2.2
- net VDIV: now also U$2.P0.18
- net VM: now also D2.C; no longer D2.1
Routing:
- net GPIO8: track 0.00 -> 20.5 mm
- net GPIO7: track 0.00 -> 18.8 mm
- net GPIO6: track 0.00 -> 17.1 mm
- net GPIO5: track 0.00 -> 15.7 mm
- net VBAT: track 54.3 -> 48.8 mm
- net VDIV: track 1.40 -> 4.38 mm
- net VBUS: track 34.2 -> 36.4 mm
- net SWDCLK: track 9.17 -> 11.3 mm, vias 0 -> 2
- net N$20: track 1.94 -> 3.51 mm
- net VCC: track 46.2 -> 44.7 mm
- net N$2: track 6.49 -> 7.05 mm

Commit message: agrego mpn
Parts:
- R4: value 220 -> 180
Routing:
- net SWDCLK: track 11.3 -> 10.4 mm
- net VBAT: track 48.8 -> 49.5 mm

Commit message: placa sin boton
Parts:
- removed C9: 0.1uF, SparkFun:0603-CAP
- removed D2: 200mA/100V/1V, SparkFun-DiscreteSemi:DIODE-1N4148
- removed D4, D5: 1A/23V/620mV, SparkFun-DiscreteSemi:SOD-323
- removed Q1: BSS84, transistor-small-signal:SOT23
- removed R10: 1, SparkFun:0603-RES
- removed R12: 100, SparkFun:0603-RES
- removed U$1: TLV703, SOT95P285X120-5N:SOT95P285X120-5N
- removed U$3: 10uf, Nordic_nRF:RESC0402_M
- removed U$4, U$5: 0.01uf, Nordic_nRF:RESC0402_M
- removed U$6, U$7: 1uf, Nordic_nRF:RESC0402_M
- removed U1: (no value), SparkFun-Sensors:QRE1113-W
- added C1: 10uf, adafruit:C0402
- added C2, C4: 0.01uf, adafruit:C0402
- added C5, C6: 1uf, adafruit:C0402
- added D6: MBR120, microbuilder:SOD-123
- added J3: 455-1750-1-ND, SparkFun-Connectors:1X03
- added Q3: DMG2305, microbuilder:SOT23-R
- added R11: 100k, adafruit:R0402
- added REG: TLV703, SOT95P285X120-5N:SOT95P285X120-5N
- added SENSOR: (no value), SparkFun-Sensors:QRE1113-W
- C3: value 10uF -> 10uf; device SparkFun-Capacitors:0805 -> adafruit:C0402
- R4: value 180 -> 680
- moved R7 11.1 mm to (8.30, 7.30), turned to 90 degrees
- moved R6 10.8 mm to (11.7, 7.30), turned to 90 degrees
- moved R13 10.5 mm to (23.1, 31.6)
- moved R1 10.3 mm to (24.7, 31.6)
- moved C3 6.44 mm to (1.80, 6.10), turned to 180 degrees
- renumbered U$2 to NRF52, U2 to DRV8835, U5 to BAT_CHAR, X2 to MICRO-USB
Connections:
- removed net N$11: NRF52.P0.19
- removed net N$12: D2.A, Q1.1, R12.2
- removed net N$13: C3.2, R10.1
- removed net N$16: NRF52.P0.22
- removed net N$28: NRF52.P0.05
- removed net N$29: NRF52.P0.10
- removed net N$5: NRF52.P0.23
- removed net RAW: Q1.3
- removed net VM: C9.2, D2.C, Q1.2, R10.2
- new net SERVO: J3.3, NRF52.P0.23
- net AIN1: now also NRF52.P0.22
- net AIN2: now also NRF52.P0.18
- net GND: now also C1.2, C2.2, C3.2, C4.2, C5.2, C6.2, J3.1, R11.1, REG.2; no longer C3.1, C9.1, R12.1, U$1.2, U$3.2, U$4.2, U$5.2, U$6.2, U$7.2
- net MODE: now also NRF52.P0.19
- net MOTOR2: now also DRV8835.3; no longer DRV8835.4
- net N$15: now also SENSOR.1; no longer U1.1
- net SENSOR: now also SENSOR.3; no longer U1.3
- net SENSOR_LED: now also SENSOR.2; no longer U1.2
- net VBAT: now also Q3.3; no longer D4.A
- net VBUS: now also D6.A, NRF52.VBUS, Q3.1, R11.2; no longer D5.A
- net VCC: now also C2.1, C4.1, C6.1, REG.5, SENSOR.4; no longer U$1.5, U$3.1, U$4.1, U$5.1, U$7.1, U1.4
- net VDIV: now also NRF52.P0.05; no longer NRF52.P0.18
- net VSUPL: now also C1.1, C3.1, C5.1, D6.C, J3.2, Q3.2, REG.1, REG.3; no longer D4.C, D5.C, U$1.1, U$1.3, U$6.1
Routing:
- net VCC: track 44.7 -> 89.6 mm, vias 2 -> 5
- net VBUS: track 36.4 -> 71.8 mm, vias 3 -> 5
- net AIN2: track 0.00 -> 32.7 mm, vias 0 -> 4
- net AIN1: track 0.00 -> 31.4 mm, vias 0 -> 2
- net VSUPL: track 13.3 -> 44.7 mm, vias 0 -> 3
- net MODE: track 0.00 -> 30.8 mm, vias 0 -> 2
- net SERVO: track 0.00 -> 21.9 mm, vias 0 -> 3
- net SENSOR: track 0.00 -> 7.65 mm, vias 0 -> 1
- net VBAT: track 49.5 -> 55.4 mm
- net N$15: track 0.00 -> 3.32 mm, vias 0 -> 1
- net VDIV: track 4.38 -> 6.69 mm
Other:
- board text added: "BAT"
- board text added: "DESIGN: SANSIL"
- board text added: "GND"
- board text added: "M30CAR"
- board text added: "MOTOR"
- board text added: "SERVO"
- board text added: "vcc"

Commit message: placa finalizada
Parts:
- added K1: TS-1188E, OPL_Switch:SW4-SMD-7.0X3.5X3.5MM-90D
- moved C1 1.50 mm to (19.3, 20.5)
- moved D6 1.43 mm to (21.5, 19.4)
- moved R11 1.40 mm to (19.3, 17.5)
Connections:
- new net VPOW: C1.1, D6.C, K1.1, Q3.2
- net GND: now also K1.S1, K1.S2
- net VSUPL: now also K1.2; no longer C1.1, D6.C, Q3.2
Routing:
- net VPOW: track 0.00 -> 24.4 mm, vias 0 -> 2
- net VSUPL: track 44.7 -> 46.8 mm, vias 3 -> 2
- net VBUS: track 71.8 -> 71.2 mm

Commit message: assemby drawing
Other:
- board size 30 x 50.1 mm -> 1.3 x 8.1 mm
- board text removed: "BAT"
- board text removed: "DESIGN: SANSIL"
- board text removed: "GND"
- board text removed: "M30CAR"
- board text removed: "MOTOR"
- board text removed: "SERVO"
- board text removed: "vcc"
