File: minM3car.sch (EAGLE design)
At the start: 38 parts, among them Q1 BSS84, U1 QRE1113SMD-W, U2 DRV8835

Commit message: nuevo avance
Parts:
- removed JP3: (no value), adafruit:PINHD-1X3
- added J1: (no value), SparkFun-Connectors:CONN_02
- R4: value 2k -> 220
Connections:
- new net GPIO1: JP1.6, U$2.P0.02
- new net GPIO2: JP1.5, U$2.P0.028
- new net GPIO3: JP1.4, U$2.P0.29
- new net GPIO4: JP1.3, U$2.P0.30
- new net LED1: R8.1, U$2.P0.03
- new net LED2: R9.1, U$2.P1.04
- new net N$11: U$2.P1.03
- new net N$14: U$2.P1.00
- new net N$16: U$2.P0.22
- new net N$17: JP2.3
- new net N$18: JP2.4
- new net N$19: U$2.P1.15
- new net N$22: U$2.P1.13
- new net N$23: U$2.P1.11
- new net N$24: JP2.5
- new net N$25: U$2.P1.02
- new net N$26: U$2.P1.01
- new net N$27: U$2.P0.04
- new net N$28: U$2.P0.05
- new net N$29: U$2.P0.10
- new net N$30: U$2.P0.31
- new net N$31: JP2.6
- net GND: now also J1.2, JP1.1
- net N$10: now also U$2.P1.06; no longer JP3.3
- net N$4: now also U$2.P0.21; no longer JP3.1
- net N$5: now also JP2.1; no longer R8.1
- net N$6: now also JP2.2; no longer R9.1
- net N$7: now also U$2.P0.09; no longer JP3.2
- net VBAT: now also J1.1
- net VCC: now also JP1.2; no longer U2.VM
- net VSUPL: now also U2.VM
Other:
- moved on the sheet: JP1, JP2

Commit message: nuevo avance
Parts:
- D2: value (none) -> 200mA/100V/1V; device SparkFun-DiscreteSemi:DIODESOD -> SparkFun-DiscreteSemi:DIODE-1N4148
- U1: value QRE1113SMD-W -> (none)
Connections:
- removed net N$14: U$2.P1.00
- removed net N$17: JP2.3
- removed net N$18: JP2.4
- removed net N$24: JP2.5
- removed net N$25: U$2.P1.02
- removed net N$26: U$2.P1.01
- removed net N$31: JP2.6
- new net GPIO5: JP2.6, U$2.P1.02
- new net GPIO6: JP2.5, U$2.P1.01
- new net GPIO7: JP2.4, U$2.P1.03
- new net GPIO8: JP2.3, U$2.P1.00
- net GND: now also JP2.1
- net N$11: now also U$2.P0.19; no longer U$2.P1.03
- net N$5: now also U$2.P0.23; no longer JP2.1
- net N$6: now also U$2.P0.12; no longer JP2.2
- net VCC: now also JP2.2
- net VDIV: now also U$2.P0.18
Changed lines of the file:
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@@
 <part name="GND3" library="SparkFun-PowerSymbols" deviceset="GND" device=""/>
 <part name="TC2" library="TagConnect" deviceset="TC2050-IDC" device="-NL"/>
-<part name="Q1" library="transistor-small-signal" library_urn="urn:adsk.eagle:library:401" deviceset="BSS84" device="" package3d_urn="urn:adsk.eagle:package:28738/2">
+<part name="Q1" library="transistor-small-signal" library_urn="urn:adsk.eagle:library:401" deviceset="BSS84" device="" package3d_urn="urn:adsk.eagle:package:29752/1">
 <attribute name="MF" value=""/>
 <attribute name="MPN" value=""/>
 <attribute name="OC_FARNELL" value="unknown"/>
 </part>
-<part name="D2" library="SparkFun-DiscreteSemi" deviceset="DIODE" device="SOD"/>
+<part name="D2" library="SparkFun-DiscreteSemi" deviceset="DIODE" device="-1N4148" value="200mA/100V/1V"/>
 <part name="R10" library="SparkFun" deviceset="RESISTOR" device="0603-RES" value="1">
 <attribute name="MF" value=""/>
@@
 </part>
 <part name="P+8" library="SparkFun" deviceset="VCC" device=""/>
-<part name="D1" library="SparkFun-LED" library_urn="urn:adsk.eagle:library:529" deviceset="LED-BLUE" device="0603" package3d_urn="urn:adsk.eagle:package:39354/1" value="BLUE"/>
-<part name="D3" library="SparkFun-LED" library_urn="urn:adsk.eagle:library:529" deviceset="LED-RED" device="0603" package3d_urn="urn:adsk.eagle:package:39354/1" value="RED"/>
+<part name="D1" library="SparkFun-LED" deviceset="LED-BLUE" device="0603" value="BLUE"/>
+<part name="D3" library="SparkFun-LED" deviceset="LED-RED" device="0603" value="RED"/>
 <part name="R8" library="adafruit" deviceset="R-US_" device="R0402" value="180"/>
 <part name="R9" library="adafruit" deviceset="R-US_" device="R0402" value="180"/>
@@
 </plain>
 <instances>
-<instance part="U1" gate="G$1" x="73.66" y="129.54" smashed="yes" rot="R180">
+<instance part="U1" gate="&gt;NAME" x="73.66" y="129.54" smashed="yes" rot="R180">
 <attribute name="NAME" x="78.994" y="134.62" size="1.778" layer="95" font="vector" rot="R270"/>
 <attribute name="VALUE" x="65.786" y="134.62" size="1.778" layer="96" font="vector" rot="R270" align="top-left"/>
@@
 <wire x1="162.56" y1="63.5" x2="154.94" y2="63.5" width="0.1524" layer="91"/>
 <label x="154.94" y="63.5" size="1.27" layer="95" rot="R180" xref="yes"/>
+</segment>
+<segment>
+<pinref part="JP2" gate="A" pin="1"/>
+<wire x1="190.5" y1="63.5" x2="182.88" y2="63.5" width="0.1524" layer="91"/>
+<label x="182.88" y="63.5" size="1.27" layer="95" rot="R180" xref="yes"/>
 </segment>
 </net>
@@
 </segment>
 <segment>
-<pinref part="U1" gate="G$1" pin="E"/>
+<pinref part="U1" gate="&gt;NAME" pin="E"/>
 <wire x1="76.2" y1="137.16" x2="76.2" y2="139.7" width="0.1524" layer="91"/>
 <pinref part="P+6" gate="VCC" pin="VCC"/>
@@
 <wire x1="162.56" y1="60.96" x2="154.94" y2="60.96" width="0.1524" layer="91"/>
 <label x="154.94" y="60.96" size="1.27" layer="95" rot="R180" xref="yes"/>
+</segment>
+<segment>
+<pinref part="JP2" gate="A" pin="2"/>
+<wire x1="190.5" y1="60.96" x2="182.88" y2="60.96" width="0.1524" layer="91"/>
+<label x="182.88" y="60.96" size="1.27" layer="95" rot="R180" xref="yes"/>
 </segment>
 </net>
@@
 <net name="SENSOR_LED" class="0">
 <segment>
-<pinref part="U1" gate="G$1" pin="K"/>
+<pinref part="U1" gate="&gt;NAME" pin="K"/>
 <wire x1="68.58" y1="137.16" x2="68.58" y2="139.7" width="0.1524" layer="91"/>
 <label x="68.58" y="139.7" size="1.4224" layer="95" rot="R180" xref="yes"/>
@@
 <net name="SENSOR" class="0">
 <segment>
-<pinref part="U1" gate="G$1" pin="C"/>
+<pinref part="U1" gate="&gt;NAME" pin="C"/>
 <wire x1="76.2" y1="124.46" x2="76.2" y2="119.38" width="0.1524" layer="91"/>
 <pinref part="R6" gate="G$1" pin="1"/>
@@
 <pinref part="R7" gate="G$1" pin="1"/>
 <wire x1="66.04" y1="119.38" x2="68.58" y2="119.38" width="0.1524" layer="91"/>
-<pinref part="U1" gate="G$1" pin="A"/>
+<pinref part="U1" gate="&gt;NAME" pin="A"/>
 <wire x1="68.58" y1="119.38" x2="68.58" y2="124.46" width="0.1524" layer="91"/>
 </segment>
@@
 <junction x="93.98" y="160.02"/>
 <label x="101.6" y="160.02" size="1.4224" layer="95" xref="yes"/>
+</segment>
+<segment>
+<pinref part="U$2" gate="G$1" pin="P0.18"/>
+<wire x1="162.56" y1="139.7" x2="157.48" y2="139.7" width="0.1524" layer="91"/>
+<label x="157.48" y="139.7" size="1.27" layer="95" rot="R180" xref="yes"/>
 </segment>
 </net>
@@
 </segment>
 </net>
-<net name="N$11" class="1">
+<net name="GPIO7" class="0">
 <segment>
 <pinref part="U$2" gate="G$1" pin="P1.03"/>
 <wire x1="223.52" y1="93.98" x2="228.6" y2="93.98" width="0.1524" layer="91"/>
-</segment>
-</net>
-<net name="N$14" class="1">
+<label x="228.6" y="93.98" size="1.27" layer="95" xref="yes"/>
+</segment>
+<segment>
+<pinref part="JP2" gate="A" pin="4"/>
+<wire x1="190.5" y1="55.88" x2="182.88" y2="55.88" width="0.1524" layer="91"/>
+<label x="182.88" y="55.88" size="1.27" layer="95" rot="R180" xref="yes"/>
+</segment>
+</net>
+<net name="GPIO8" class="0">
 <segment>
 <pinref part="U$2" gate="G$1" pin="P1.00"/>
 <wire x1="223.52" y1="88.9" x2="228.6" y2="88.9" width="0.1524" layer="91"/>
+<label x="228.6" y="88.9" size="1.27" layer="95" xref="yes"/>
+</segment>
+<segment>
+<pinref part="JP2" gate="A" pin="3"/>
+<wire x1="190.5" y1="58.42" x2="182.88" y2="58.42" width="0.1524" layer="91"/>
+<label x="182.88" y="58.42" size="1.27" layer="95" rot="R180" xref="yes"/>
 </segment>
 </net>
@@
 </segment>
 </net>
-<net name="GPIO1" class="1">
+<net name="GPIO1" class="0">
 <segment>
 <pinref part="U$2" gate="G$1" pin="P0.02"/>
@@
 </segment>
 </net>
-<net name="N$25" class="1">
+<net name="GPIO5" class="0">
 <segment>
 <pinref part="U$2" gate="G$1" pin="P1.02"/>
 <wire x1="223.52" y1="104.14" x2="228.6" y2="104.14" width="0.1524" layer="91"/>
-</segment>
-</net>
-<net name="N$26" class="1">
+<label x="228.6" y="104.14" size="1.27" layer="95" xref="yes"/>
+</segment>
+<segment>
+<pinref part="JP2" gate="A" pin="6"/>
+<wire x1="190.5" y1="50.8" x2="182.88" y2="50.8" width="0.1524" layer="91"/>
+<label x="182.88" y="50.8" size="1.27" layer="95" rot="R180" xref="yes"/>
+</segment>
+</net>
+<net name="GPIO6" class="0">
 <segment>
 <pinref part="U$2" gate="G$1" pin="P1.01"/>
 <wire x1="223.52" y1="99.06" x2="228.6" y2="99.06" width="0.1524" layer="91"/>
+<label x="228.6" y="99.06" size="1.27" layer="95" xref="yes"/>
+</segment>
+<segment>
+<pinref part="JP2" gate="A" pin="5"/>
+<wire x1="190.5" y1="53.34" x2="182.88" y2="53.34" width="0.1524" layer="91"/>
+<label x="182.88" y="53.34" size="1.27" layer="95" rot="R180" xref="yes"/>
 </segment>
 </net>
@@
 </segment>
 </net>
-<net name="GPIO2" class="1">
+<net name="GPIO2" class="0">
 <segment>
 <pinref part="U$2" gate="G$1" pin="P0.028"/>
@@
 </segment>
 </net>
-<net name="GPIO3" class="1">
+<net name="GPIO3" class="0">
 <segment>
 <pinref part="U$2" gate="G$1" pin="P0.29"/>
@@
 </segment>
 </net>
-<net name="GPIO4" class="1">
+<net name="GPIO4" class="0">
 <segment>
 <pinref part="U$2" gate="G$1" pin="P0.30"/>
@@
 </segment>
 </net>
-<net name="N$5" class="1">
-<segment>
-<pinref part="JP2" gate="A" pin="1"/>
-<wire x1="190.5" y1="63.5" x2="182.88" y2="63.5" width="0.1524" layer="91"/>
-</segment>
-</net>
-<net name="N$6" class="1">
-<segment>
-<pinref part="JP2" gate="A" pin="2"/>
-<wire x1="190.5" y1="60.96" x2="182.88" y2="60.96" width="0.1524" layer="91"/>
-</segment>
-</net>
-<net name="N$17" class="1">
-<segment>
-<pinref part="JP2" gate="A" pin="3"/>
-<wire x1="190.5" y1="58.42" x2="182.88" y2="58.42" width="0.1524" layer="91"/>
-</segment>
-</net>
-<net name="N$18" class="1">
-<segment>
-<pinref part="JP2" gate="A" pin="4"/>
-<wire x1="190.5" y1="55.88" x2="182.88" y2="55.88" width="0.1524" layer="91"/>
-</segment>
-</net>
-<net name="N$24" class="1">
-<segment>
-<pinref part="JP2" gate="A" pin="5"/>
-<wire x1="190.5" y1="53.34" x2="182.88" y2="53.34" width="0.1524" layer="91"/>
-</segment>
-</net>
-<net name="N$31" class="1">
-<segment>
-<pinref part="JP2" gate="A" pin="6"/>
-<wire x1="190.5" y1="50.8" x2="182.88" y2="50.8" width="0.1524" layer="91"/>
-</segment>
-</net>
+<net name="N$5" class="0">
+<segment>
+<pinref part="U$2" gate="G$1" pin="P0.23"/>
+<wire x1="162.56" y1="124.46" x2="157.48" y2="124.46" width="0.1524" layer="91"/>
+</segment>
+</net>
+<net name="N$6" class="0">
+<segment>
+<pinref part="U$2" gate="G$1" pin="P0.12"/>
+<wire x1="162.56" y1="119.38" x2="157.48" y2="119.38" width="0.1524" layer="91"/>
+</segment>
+</net>
+<net name="N$11" class="0">
+<segment>
+<pinref part="U$2" gate="G$1" pin="P0.19"/>
+<wire x1="162.56" y1="134.62" x2="157.48" y2="134.62" width="0.1524" layer="91"/>
+</segment>
+</net>

Commit message: agrego mpn
Parts:
- D1, D3: MPN (none) -> 150060YS75000
- D4, D5: MPN (none) -> BAT20JFILM
- R1, R13: MPN (none) -> RC0402JR-07100KL
- R2, R3: LINK (none) -> https://www.seeedstudio.com/opl.html; MPN (none) -> BLM15BB220SN1D
- R4: value 220 -> 180; LINK (none) -> https://www.seeedstudio.com/opl.html; MPN (none) -> RC0402FR-07180RL
- R5: MPN (none) -> RC0402FR-072KL
- R6: LINK (none) -> https://www.seeedstudio.com/opl.html; MPN (none) -> RC0402JR-0710KL
- R7: MPN (none) -> 0402WGF2000TCE
- R8, R9: LINK (none) -> https://www.seeedstudio.com/opl.html; MPN (none) -> RC0402FR-07180RL
- U$1: LINK (none) -> https://uy.mouser.com/ProductDetail/Texas-Instruments/TLV70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; MPN (none) -> TLV7031DBVR
- U$3: MPN (none) -> GRM155R60J106ME44D
- U$4, U$5: MPN (none) -> CL05C100JB5NNNC
- U$6, U$7: MPN (none) -> CL05A105KP5NNNC
- U1: LINK (none) -> https://uy.mouser.com/ProductDetail/ON-Semiconductor-Fairch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; MPN (none) -> QRE1113GR
- U2: LINK (none) -> https://uy.mouser.com/ProductDetail/Texas-Instruments/DRV88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; MPN (none) -> DRV8835DSSR
- U5: LINK (none) -> https://uy.mouser.com/ProductDetail/Microchip-Technology/MC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; MPN (none) -> MCP73831T-2ACI/OT
- X2: LINK (none) -> https://www.digikey.com/product-detail/en/amphenol-icc-fci/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; MPN (none) -> 10103592-0001LF

Commit message: placa sin boton
Parts:
- removed C9: 0.1uF, SparkFun:CAP0603-CAP
- removed D2: 200mA/100V/1V, SparkFun-DiscreteSemi:DIODE-1N4148
- removed D4, D5: 1A/23V/620mV, SparkFun-DiscreteSemi:DIODE-SCHOTTKY-BAT20J
- removed Q1: BSS84, transistor-small-signal:BSS84
- removed R10: 1, SparkFun:RESISTOR0603-RES
- removed R12: 100, SparkFun:RESISTOR0603-RES
- removed U$3: 10uf, Nordic_nRF:CAPACITOR_0402_M
- removed U$4, U$5: 0.01uf, Nordic_nRF:CAPACITOR_0402_M
- removed U$6, U$7: 1uf, Nordic_nRF:CAPACITOR_0402_M
- added C1: 10uf, adafruit:C-USC0402
- added C2, C4: 0.01uf, adafruit:C-USC0402
- added C5, C6: 1uf, adafruit:C-USC0402
- added D6: MBR120, microbuilder:DIODE-SCHOTTKYSOD-123
- added J3: 455-1750-1-ND, SparkFun-Connectors:CONN_03
- added Q3: DMG2305, microbuilder:MOSFET-P
- added R11: 100k, adafruit:R-US_R0402
- C3: value 10uF -> 10uf; device SparkFun-Capacitors:CAP0805 -> adafruit:C-USC0402; OC_FARNELL unknown -> (none); PARTN (none) -> GRM155R60G106ME44D
- NRF52: MPN (none) -> 113990556
- R4: value 180 -> 680; MPN RC0402FR-07180RL -> RC0402JR-07680RL
- renumbered U$1 to REG, U$2 to NRF52, U1 to SENSOR, U2 to DRV8835, U5 to BAT_CHAR, X2 to MICRO-USB
Connections:
- removed net N$11: NRF52.P0.19
- removed net N$12: D2.A, Q1.G, R12.2
- removed net N$13: C3.2, R10.1
- removed net N$16: NRF52.P0.22
- removed net N$28: NRF52.P0.05
- removed net N$29: NRF52.P0.10
- removed net N$5: NRF52.P0.23
- removed net RAW: Q1.D
- removed net VM: C9.2, D2.C, Q1.S, R10.2
- new net SERVO: J3.3, NRF52.P0.23
- net AIN1: now also NRF52.P0.22
- net AIN2: now also NRF52.P0.18
- net GND: now also C1.2, C2.2, C3.2, C4.2, C5.2, C6.2, J3.1, R11.1; no longer C3.1, C9.1, R12.1, U$3.2, U$4.2, U$5.2, U$6.2, U$7.2
- net MODE: now also NRF52.P0.19
- net MOTOR2: now also DRV8835.AOUT2; no longer DRV8835.BOUT1
- net VBAT: now also Q3.D; no longer D4.A
- net VBUS: now also D6.A, NRF52.VBUS, Q3.G, R11.2; no longer D5.A
- net VCC: now also C2.1, C4.1, C6.1; no longer U$3.1, U$4.1, U$5.1, U$7.1
- net VDIV: now also NRF52.P0.05; no longer NRF52.P0.18
- net VSUPL: now also C1.1, C3.1, C5.1, D6.C, J3.2, Q3.S; no longer D4.C, D5.C, U$6.1
Other:
- note removed: "VM"
- moved on the sheet: C3

Commit message: placa finalizada
Parts:
- added K1: TS-1188E, OPL_Switch:SMD-BUTTON(2+2P-7X3.5MM-90D)
- C1, C10, C3: MPN (none) -> GRM155R60G106ME44D; PARTN GRM155R60G106ME44D -> (none)
- C2, C4: MPN (none) -> CL05C100JB5NNNC; PARTN CL05C100JB5NNNC -> (none)
- C5, C6: MPN (none) -> CL05A105KP5NNNC; PARTN CL05A105KP5NNNC -> (none)
- LED1: MPN (none) -> 150060GS75000; PARTN 150060GS75000 -> (none)
Connections:
- new net VPOW: C1.1, D6.C, K1.1, Q3.S
- net GND: now also K1.S1, K1.S2
- net VSUPL: now also K1.2; no longer C1.1, D6.C, Q3.S
